Commit message: holy started to walk

File: src/bioloid_interface/urdf/TypeA.urdf.xacro (robot description, xacro)
@@ -20,5 +20,5 @@
             <origin rpy="${pi_half} 0 0" xyz="${reflect*0.070} 0 0.03"/>
             <axis xyz="${reflect} 0 0"/>
-            <limit effort="1000.0" lower="-${pi}" upper="${pi}" velocity="0.5"/>
+            <limit effort="1000.0" lower="-${pi}" upper="${pi}" velocity="1.0"/>
         </joint>
         <link name="${prefix}_upper_arm">
@@ -38,5 +38,5 @@
 	    <origin rpy="0 ${reflect*-1.5} 0" xyz="0.00 0 0.0"/>
 	    <axis xyz="0 -1 0"/>
-	    <limit effort="1000.0" lower="-3.14" upper="3.14" velocity="0.5"/>
+	    <limit effort="1000.0" lower="-3.14" upper="3.14" velocity="1.0"/>
 	  </joint>
         <link name="${prefix}_forearm">
@@ -54,5 +54,5 @@
 	    <origin rpy="0 0 0" xyz="0.00 0 -0.08"/>
 	    <axis xyz="0 -1 0"/>
-	    <limit effort="1000.0" lower="-3.14" upper="3.14" velocity="0.5"/>
+	    <limit effort="1000.0" lower="-3.14" upper="3.14" velocity="1.0"/>
 	  </joint>
     </xacro:macro>
@@ -74,5 +74,5 @@
 	        <origin rpy="0 0 0" xyz="${reflect*0.030} 0 -0.06"/>
 	        <axis xyz="0 0 -1"/>
-	        <limit effort="1000.0" lower="-0.5" upper="0.5" velocity="0.5"/>
+	        <limit effort="1000.0" lower="-0.5" upper="0.5" velocity="1.0"/>
         </joint>
         <link name="${prefix}_hip_split">
@@ -92,5 +92,5 @@
             <origin rpy="0 0 0" xyz="0 0 0"/>
             <axis xyz="0 1 0"/>
-            <limit effort="1000.0" lower="-1.0" upper="1.0" velocity="0.5"/>
+            <limit effort="1000.0" lower="-1.0" upper="1.0" velocity="1.0"/>
         </joint>
         <link name="${prefix}_upper_leg">
@@ -108,5 +108,5 @@
             <origin rpy="0 0 0" xyz="0 0 0"/>
             <axis xyz="${reflect*-1} 0 0"/>
-            <limit effort="1000.0" lower="-${pi}" upper="${pi}" velocity="0.5"/>
+            <limit effort="1000.0" lower="-${pi}" upper="${pi}" velocity="1.0"/>
         </joint>
         <link name="${prefix}_calf">
@@ -124,5 +124,5 @@
             <origin rpy="0 0 0" xyz="0 0 -0.08"/>
             <axis xyz="${reflect*1} 0 0"/>
-            <limit effort="1000.0" lower="-${pi}" upper="${pi}" velocity="0.5"/>
+            <limit effort="1000.0" lower="-${pi}" upper="${pi}" velocity="1.0"/>
         </joint>
         <link name="${prefix}_foot">
@@ -140,5 +140,5 @@
             <origin rpy="0 0 0" xyz="0 0 -0.045"/>
             <axis xyz="${reflect} 0 0"/>
-            <limit effort="1000.0" lower="-${pi}" upper="${pi}" velocity="0.5"/>
+            <limit effort="1000.0" lower="-${pi}" upper="${pi}" velocity="1.0"/>
         </joint>
         <link name="${prefix}_foot_pad">
@@ -156,5 +156,5 @@
             <origin rpy="0 0 0" xyz="0 0 -0.03"/>
             <axis xyz="0 -1 0"/>
-            <limit effort="1000.0" lower="-${pi}" upper="${pi}" velocity="0.5"/>
+            <limit effort="1000.0" lower="-${pi}" upper="${pi}" velocity="1.0"/>
         </joint>
     </xacro:macro>
