Commit message: ikfast leg plugins work

File: src/holy_controllers/urdf/TypeA.urdf.xacro (robot description, xacro)
@@ -124,5 +124,6 @@
             <origin rpy="0 0 0" xyz="0 0 -0.08"/>
             <axis xyz="${reflect*1} 0 0"/>
-            <limit effort="1000.0" lower="-${pi}" upper="${pi}" velocity="1.0"/>
+            <!-- <limit effort="1000.0" lower="-${pi}" upper="${pi}" velocity="1.0"/> -->
+	    <limit effort="1000.0" lower="-0.1" upper="${pi}" velocity="1.0"/>
         </joint>
         <link name="${prefix}_foot">

Commit message: urdf file with correct joint limits

File: src/holy_controllers/urdf/TypeA.urdf.xacro (robot description, xacro)
@@ -124,6 +124,5 @@
             <origin rpy="0 0 0" xyz="0 0 -0.08"/>
             <axis xyz="${reflect*1} 0 0"/>
-            <!-- <limit effort="1000.0" lower="-${pi}" upper="${pi}" velocity="1.0"/> -->
-	    <limit effort="1000.0" lower="-0.1" upper="${pi}" velocity="1.0"/>
+            <limit effort="1000.0" lower="-${pi}" upper="${pi}" velocity="1.0"/>
         </joint>
         <link name="${prefix}_foot">
