Commit message: modified URDF to reflect new reinforced hardware/mechanics configuration. Fixed Moveit Setup Assistant looking for bioloid_interface. Initialization of holy produces the Error "Parameter '~moveit_controller_manager' not specified. This is needed to identify the plugin to use for interacting with controllers. No paths can be executed.", which means the project doesn't work right now :(

File: src/holy_controllers/urdf/holy.urdf (robot description, URDF)
Before this commit: robot awesome-o, 19 links, 18 joints
Links:
- link L_hip: geometry visual box size=0.0725 0.04 0.03
- link R_hip: geometry visual box size=0.0725 0.04 0.03
Joints:
- joint L_HAA: origin xyz=-0.03 0 -0.06 rpy=0 0 0 -> xyz=-0.0475 0 -0.06 rpy=0 0 0
- joint R_HAA: origin xyz=0.03 0 -0.06 rpy=0 0 0 -> xyz=0.0475 0 -0.06 rpy=0 0 0

Commit message: walking laeuft

File: src/holy_controllers/urdf/holy.urdf (robot description, URDF)
Before this commit: robot awesome-o, 19 links, 18 joints
Joints:
- joint L_HR: limit lower=-0.9940195505 upper=1.4603497101 effort=1000.0 velocity=1.0 -> lower=-1.0246991663 upper=1.4296700943 effort=1000.0 velocity=1.0
- joint R_HFE: limit lower=-2.712078033 upper=0.7240389319 effort=1000.0 velocity=1.0 -> lower=-2.8041168803 upper=0.6320000846 effort=1000.0 velocity=1.0
